File: keyborad.sch (KiCad schematic (older format))
At the start: 21 parts, among them SW1 SW_DIP_x01, SW2 SW_DIP_x01, SW3 SW_DIP_x01, SW4 SW_DIP_x01, SW5 SW_DIP_x01, SW6 SW_DIP_x01

Commit message: ちまちま修正
いらないファイルたちは消した
Parts:
- removed H3, H4, H5, H6, H7, H8, H9: hole, Pin_Headers:Pin_Header_Straight_1x01_Pitch1.27mm, symbol hole
- added P1, P10, P11, P12, P13, P2, P3, P4, P5, P6, P7, P8, P9: 1pin, Pin_Headers:Pin_Header_Straight_1x01_Pitch1.27mm, symbol 1pin
Connections:
- net col0: now also P1.1, P8.1
- net col1: now also P2.1, P9.1
- net col2: now also P10.1, P3.1
- net col3: now also P11.1, P4.1
- net col4: now also P12.1, P5.1
- net col5: now also P13.1, P6.1
- net row0: now also P7.1
